File: usb3_3v.kicad_pcb (KiCad board)
At the start: 2 copper layers, 6 parts, among them J1 USB-MICRO-B, P1 +3.3, P2 GND, U1 AAT3221 / MIC5504

Commit message: - pcb done, add gerbers
Parts:
- added D1: LED, SM0603, F.Cu at (227.3, 141.6)
- added R1: 1K, SM0402_r, F.Cu at (224.3, 140.7)
- moved C1 10.9 mm to (221.0, 142.2)
- moved C2 8.92 mm to (224.3, 142.2), turned to 180 degrees
- moved P2 2.54 mm to (232.4, 146.1), turned to 270 degrees
- moved U1 1.27 mm to (222.2, 144.8)
- turned P1 to 270 degrees
Connections:
- C1 pad 1: GND -> /+5v
- J1 pad 1: GND -> /+5v
- U1 pad 1: GND -> /+5v
- U1 pad 2: (no net) -> GND
- U1 pad 3: GND -> /+5v
Routing:
- net /+3.3v: track 0.00 -> 11.5 mm
- net /+5v: track 0.00 -> 10.1 mm
- added copper zone on B.Cu, net GND
- added copper zone on F.Cu, net GND
Other:
- board outline added: 20.8 x 11.2 mm
- board text added: "github.com/ noahp/usb3_3v v0.1"

Commit message: - fix gerbers
Routing:
- net N-000007: track 0.00 -> 2.65 mm
Changed lines of the file:
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@@
   (general
     (links 19)
-    (no_connects 5)
+    (no_connects 4)
     (area 211.767 139.141999 235.339 150.418001)
     (thickness 1.6)
     (drawings 9)
-    (tracks 17)
+    (tracks 19)
     (zones 0)
     (modules 8)
@@
     (visible_elements 7FFFFFBF)
     (pcbplotparams
-      (layerselection 15761409)
+      (layerselection 284196865)
       (usegerberextensions true)
       (excludeedgelayer true)
@@
   (gr_arc (start 233.426 139.7) (end 233.426 139.192) (angle 90) (layer Edge.Cuts) (width 0.1))
   (gr_arc (start 213.614 139.7) (end 213.106 139.7) (angle 90) (layer Edge.Cuts) (width 0.1))
-  (segment (start 230.82 143.83) (end 232.09 143.83) (width 0.254) (layer F.Cu) (net 1) (status 800000))
+  (segment (start 230.82 143.83) (end 232.09 143.83) (width 0.254) (layer F.Cu) (net 1))
   (segment (start 225.806 143.83) (end 230.82 143.83) (width 0.254) (layer F.Cu) (net 1))
-  (segment (start 232.09 143.83) (end 232.41 143.51) (width 0.254) (layer F.Cu) (net 1) (status C00000))
+  (segment (start 232.09 143.83) (end 232.41 143.51) (width 0.254) (layer F.Cu) (net 1))
   (segment (start 224.75 143.83) (end 225.806 143.83) (width 0.254) (layer F.Cu) (net 1))
   (segment (start 225.806 143.83) (end 225.867 143.83) (width 0.254) (layer F.Cu) (net 1))
@@
   (segment (start 220.345 143.48) (end 221.9 143.48) (width 0.254) (layer F.Cu) (net 2))
   (segment (start 221.9 143.48) (end 222.25 143.83) (width 0.254) (layer F.Cu) (net 2))
+  (segment (start 227.33 140.843) (end 227.203 140.716) (width 0.254) (layer F.Cu) (net 4) (status C00000))
+  (segment (start 227.203 140.716) (end 224.73158 140.716) (width 0.254) (layer F.Cu) (net 4) (status C00000))
   (zone (net 3) (net_name GND) (layer F.Cu) (hatch edge 0.508)
     (connect_pads (clearance 0.254))
